File: spark!2350.kicad_sch (KiCad schematic)
At the start: 22 parts, among them J1 USB_C_Receptacle_USB2.0_16P, J2 LIPO, U1 RP2350_80QFN, U2 <value>, U3 MCP73871, U4 MCP1700x-330xxTT, U5 W25Q128JVS

Commit message: i kinda forgot to bump hardware files regularly so here ya go!
Parts:
- removed J2: LIPO, Connector_JST:JST_PH_S2B-PH-K_1x02_P2.00mm_Horizontal, symbol Connector:Conn_01x02_Socket
- added C10, C11, C12, C13, C14, C15, C16, C17, C18, C8, C9: 100n, RP2350_80QFN_minimal:C_0402_1005Metric_small_pads, symbol Device:C_45deg
- added C19: 4.7u, RP2350_80QFN_minimal:C_0402_1005Metric_small_pads, symbol Device:C_45deg
- added C20: 100n, RP2350_80QFN_minimal:C_0402_1005Metric_small_pads, symbol Device:C
- added C21, C22: 15p, RP2350_80QFN_minimal:C_0402_1005Metric_small_pads, symbol Device:C
- added D1: Red, LED_SMD:LED_0805_2012Metric, symbol Device:LED_Small
- added D2: Green, LED_SMD:LED_0805_2012Metric, symbol Device:LED_Small
- added D3: SK6812MINI, LED_SMD:LED_SK6812MINI_PLCC4_3.5x3.5mm_P1.75mm, symbol LED:SK6812MINI
- added J3: Left, castellated:27right, symbol Connector:Conn_01x28_Socket
- added J4: Right, castellated:27left, symbol Connector:Conn_01x28_Socket
- added JP2: SolderJumper_2_Bridged, Jumper:SolderJumper-2_P1.3mm_Bridged_RoundedPad1.0x1.5mm, symbol Jumper:SolderJumper_2_Bridged
- added L1: 3.3u, RP2350_80QFN_minimal:L_pol_2016, symbol Device:L
- added R10, R11: 200, Resistor_SMD:R_0402_1005Metric, symbol Device:R_Small
- added R12, R13: 27, Resistor_SMD:R_0402_1005Metric, symbol Device:R_Small
- added R14: 0, Resistor_SMD:R_0402_1005Metric, symbol Device:R_Small
- added R15, R19, R8: 10k, Resistor_SMD:R_0402_1005Metric, symbol Device:R_Small
- added R16, R17: 1k, Resistor_SMD:R_0402_1005Metric, symbol Device:R_Small
- added R18: 470, Resistor_SMD:R_0402_1005Metric, symbol Device:R_Small
- added R20, R21: 5.1k, Resistor_SMD:R_0402_1005Metric, symbol Device:R_Small
- added R9: 100k, Resistor_SMD:R_0402_1005Metric, symbol Device:R_Small
- added SW1: BOOT, TS-1088-AR02016:SW_TS-1088-AR02016, symbol Switch:SW_Push
- added SW2: RUN, TS-1088-AR02016:SW_TS-1088-AR02016, symbol Switch:SW_Push
- added Y1: ABM8-272-T3, footprints:ABM8-272-T3_ABR, symbol Device:Crystal_GND24
- C1: value 10uF -> 10u; footprint (none) -> RP2350_80QFN_minimal:C_0402_1005Metric_small_pads; LCSC (none) -> C15525
- C2: value 4.7uF -> 4.7u; footprint (none) -> RP2350_80QFN_minimal:C_0402_1005Metric_small_pads; LCSC (none) -> C29823
- C3, C4: value 1uF -> 1u; footprint (none) -> RP2350_80QFN_minimal:C_0402_1005Metric_small_pads; LCSC (none) -> C52923
- C5, C6, C7: footprint (none) -> RP2350_80QFN_minimal:C_0402_1005Metric_small_pads; LCSC (none) -> C29823
- J1: footprint Connector_USB:USB_C_Receptacle_GCT_USB4085 -> Connector_USB:USB_C_Receptacle_HRO_TYPE-C-31-M-12; LCSC (none) -> C165948
- JP1: footprint Jumper:SolderJumper-2_P1.3mm_Open_TrianglePad1.0x1.5mm -> Jumper:SolderJumper-2_P1.3mm_Open_RoundedPad1.0x1.5mm; now not fitted
- R1, R3, R4, R5, R6: footprint (none) -> Resistor_SMD:R_0402_1005Metric; LCSC (none) -> C25744
- R2: footprint (none) -> Resistor_SMD:R_0402_1005Metric; LCSC (none) -> C25890
- R7: footprint (none) -> Resistor_SMD:R_0402_1005Metric; LCSC (none) -> C25105
- U1: LCSC (none) -> C42415655
- U2: footprint (none) -> RM2:rpi_rmc20452t
- U3: LCSC (none) -> C511310
- U4: LCSC (none) -> C39051
- U5: LCSC (none) -> C97521
Connections:
- net +1V1: now also U1.10 (DVDD), U1.32 (DVDD), U1.51 (DVDD), C17.2, C18.2, C19.2, L1.1
- net +3V3: now also U1.15 (IOVDD), U1.24 (IOVDD), U1.29 (IOVDD), U1.41 (IOVDD), U1.5 (IOVDD), U1.50 (IOVDD), U1.59 (ADC_AVDD), U1.60 (IOVDD), U1.68 (USB_OTP_VDD), U1.69 (QSPI_IOVDD), U1.76 (IOVDD), U2.14 (VDDIO), U2.16 (VIN), U5.8 (VCC), C10.2, C11.2, C12.2, C13.2, C14.2, C15.2, C16.2, C20.1, C8.2, C9.2, D3.4 (VDD), J4.2 (Pin_2), R10.2, R11.2, R15.1
- net GND: now also J1.A1 (GND), J1.A12 (GND), J1.B1 (GND), J1.B12 (GND), J1.S1 (SHIELD), R3.1, R5.1, U2.1 (GND), U2.11 (GND), U2.15 (GND), U2.21 (GND), U2.4 (GND), U2.7 (GND), U5.4 (GND), C10.1, C11.1, C12.1, C13.1, C14.1, C15.1, C16.1, C17.1, C18.1, C19.1, C20.2, C21.1, C22.1, C8.1, C9.1, D3.2 (VSS), J3.1 (Pin_1), J4.1 (Pin_1), R20.2, R21.2, R9.1, SW1.1, SW2.1, Y1.2, Y1.4; no longer R3.2, R5.2
- net VBUS: now also U3.2 (VPCC), R8.1; no longer U3.4 (PROG2)
- net VREG_LX: now also L1.2
- net at U3.9 (~{TE}): now also R5.2; no longer R5.1
- net 4: now reaches U1.1 (GPIO4)
- net 4: now also J3.8 (Pin_8)
- net 12: now reaches U1.11 (GPIO12)
- net 12: now also J3.16 (Pin_16)
- net 13: now reaches U1.12 (GPIO13)
- net 13: now also J3.17 (Pin_17)
- net 14: now reaches U1.13 (GPIO14)
- net 14: now also J3.18 (Pin_18)
- net 15: now reaches U1.14 (GPIO15)
- net 15: now also J3.19 (Pin_19)
- net 16: now reaches U1.16 (GPIO16)
- net 16: now also J3.20 (Pin_20)
- net 17: now reaches U1.17 (GPIO17)
- net 17: now also J3.21 (Pin_21)
- net 18: now reaches U1.18 (GPIO18)
- net 18: now also J3.22 (Pin_22)
- net 19: now reaches U1.19 (GPIO19)
- net 19: now also J3.23 (Pin_23)
- net 5: now reaches U1.2 (GPIO5)
- net 5: now also J3.9 (Pin_9)
- net 20: now reaches U1.20 (GPIO20)
- net 20: now also J3.24 (Pin_24)
- net 21: now reaches U1.21 (GPIO21)
- net 21: now also J3.25 (Pin_25)
- net 22: now reaches U1.22 (GPIO22)
- net 22: now also J3.26 (Pin_26)
- net 23: now reaches U1.23 (GPIO23)
- net 23: now also U2.12 (WL_ON), U2.13 (BT_ON), J3.27 (Pin_27)
- net 24: now reaches U1.25 (GPIO24)
- net 24: now also U2.5 (DI), J3.28 (Pin_28), R18.1, R19.1
- net 25: now reaches U1.26 (GPIO25)
- net 25: now also U2.9 (CS), J4.28 (Pin_28)
- net 26: now reaches U1.27 (GPIO26)
- net 26: now also J4.27 (Pin_27)
- net 27: now reaches U1.28 (GPIO27)
- net 27: now also J4.26 (Pin_26)
- net 6: now reaches U1.3 (GPIO6)
- net 6: now also J3.10 (Pin_10)
- net at U1.30 (XIN): now also C21.2, Y1.1
- net at U1.31 (XOUT): now also R17.2
- net RUN: now reaches U1.35 (RUN)
- net RUN: now also J4.5 (Pin_5), SW2.2
- net 28: now reaches U1.36 (GPIO28)
- net 28: now also J4.25 (Pin_25)
- net 29: now reaches U1.37 (GPIO29)
- net 29: now also U2.3 (SCLK), J4.24 (Pin_24)
- net 30: now reaches U1.38 (GPIO30)
- net 30: now also J4.23 (Pin_23)
- net 31: now reaches U1.39 (GPIO31)
- net 31: now also J4.22 (Pin_22)
- net 7: now reaches U1.4 (GPIO7)
- net 7: now also J3.11 (Pin_11)
- net 32: now reaches U1.40 (GPIO32)
- net 32: now also J4.21 (Pin_21)
- net 33: now reaches U1.42 (GPIO33)
- net 33: now also J4.20 (Pin_20)
- net 34: now reaches U1.43 (GPIO34)
- net 34: now also J4.19 (Pin_19)
- net 35: now reaches U1.44 (GPIO35)
- net 35: now also J4.18 (Pin_18)
- net 36: now reaches U1.45 (GPIO36)
- net 36: now also J4.17 (Pin_17)
- net 37: now reaches U1.46 (GPIO37)
- net 37: now also J4.16 (Pin_16)
- net 38: now reaches U1.47 (GPIO38)
- net 38: now also J4.15 (Pin_15)
- net 39: now reaches U1.48 (GPIO39)
- net 39: now also J4.14 (Pin_14)
- net 40: now reaches U1.49 (GPIO40_ADC0)
- net 40: now also J4.13 (Pin_13)
- net 41: now reaches U1.52 (GPIO41_ADC1)
- net 41: now also J4.12 (Pin_12)
- net 42: now reaches U1.53 (GPIO42_ADC2)
- net 42: now also J4.11 (Pin_11)
- net 43: now reaches U1.54 (GPIO43_ADC3)
- net 43: now also J4.10 (Pin_10)
- net 44: now reaches U1.55 (GPIO44_ADC4)
- net 44: now also J4.9 (Pin_9)
- net 45: now reaches U1.56 (GPIO45_ADC5)
- net 45: now also J4.8 (Pin_8)
- net 46: now reaches U1.57 (GPIO46_ADC6)
- net 46: now also J4.7 (Pin_7)
- net 47: now reaches U1.58 (GPIO47_ADC7)
- net 47: now also J4.6 (Pin_6)
- net 8: now reaches U1.6 (GPIO8)
- net 8: now also J3.12 (Pin_12)
- net 9: now reaches U1.7 (GPIO9)
- net 9: now also J3.13 (Pin_13)
- net QSPI_SD3: now reaches U1.70 (QSPI_SD3)
- net QSPI_SD3: now also U5.7 (~{HOLD}/~{RESET}/IO_{3})
- net QSPI_SCLK: now reaches U1.71 (QSPI_SCLK)
- net QSPI_SCLK: now also U5.6 (CLK)
- net QSPI_SD0: now reaches U1.72 (QSPI_SD0)
- net QSPI_SD0: now also U5.5 (DI/IO_{0})
- net QSPI_SD2: now reaches U1.73 (QSPI_SD2)
- net QSPI_SD2: now also U5.3 (~{WP}/IO_{2})
- net QSPI_SD1: now reaches U1.74 (QSPI_SD1)
- net QSPI_SD1: now also U5.2 (DO/IO_{1})
- net QSPI_SS: now reaches U1.75 (QSPI_SS)
- net QSPI_SS: now also R14.1, R16.1
- net 0: now reaches U1.77 (GPIO0)
- net 0: now also J3.4 (Pin_4), JP2.1 (A)
- net 1: now reaches U1.78 (GPIO1)
- net 1: now also J3.5 (Pin_5)
- net 2: now reaches U1.79 (GPIO2)
- net 2: now also J3.6 (Pin_6)
- net 10: now reaches U1.8 (GPIO10)
- net 10: now also J3.14 (Pin_14)
- net 3: now reaches U1.80 (GPIO3)
- net 3: now also J3.7 (Pin_7)
- net 11: now reaches U1.9 (GPIO11)
- net 11: now also J3.15 (Pin_15)
- net at U3.12 (PROG3): now also R9.2
- net +BATT: now reaches C2.1, U3.14 (V_{BAT}), U3.15 (V_{BAT}), U3.16 (V_{BAT_SENSE})
- net +BATT: now also J3.2 (Pin_2), J3.3 (Pin_3)
- net at U3.5 (THERM): now also R3.2; no longer R3.1
- net at U3.7 (STAT2): now also D2.1 (K)
- net at U3.8 (STAT1/~{LBO}): now also D1.1 (K)
- net at U5.1 (~{CS}): now also R14.2, R15.2
- net at U2.10 (nIRQ): now also R19.2
- net at U2.6 (DO): now also R18.2
- net at J1.A5 (CC1): now also R20.1
- net at J1.B5 (CC2): now also R21.1
- net DM- renamed DM -
- net DM -: now also J4.4 (Pin_4), R13.2; no longer U1.66 (USB_DM)
- net DP+ renamed DP +
- net DP +: now also J4.3 (Pin_3), R12.2; no longer U1.67 (USB_DP)
- new net: R16.2, SW1.2
- new net: R13.1, U1.66 (USB_DM)
- new net: R12.1, U1.67 (USB_DP)
- new net: C22.2, R17.1, Y1.3
- new net: R8.2, U3.4 (PROG2)
- new net: D3.3 (DIN), JP2.2 (B)
- new net: D2.2 (A), R11.1
- new net: D1.2 (A), R10.1
- no-connect marks 0 -> 2
Other:
- note removed: "TODO: Inductor"
- moved on the sheet: C3, C4, C5, C6, C7, R3, R5, R6, R7, U1, U2, U4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
